File: PCB tah les ouf.kicad_pcb (KiCad board)
At the start: 2 copper layers, 60 x 60 mm, 11 parts, among them J1 USB_C_Receptacle_USB2.0_16P, U1 ESP32-S3-WROOM-1, U2 TMC2209_SILENTSTEPSTICK, U3 TMC2209_SILENTSTEPSTICK, U4 TMC2209_SILENTSTEPSTICK, U5 TMC2209_SILENTSTEPSTICK, U6 D3V3XA4B10LP, U7 AMS1117-3.3 (UMW)

Commit message: Suppression TMC2209 x1
Parts:
- removed U5: TMC2209_SILENTSTEPSTICK, TMC2209:MODULE_TMC2209_SILENTSTEPSTICK
- added ADD1: Conn_01x04_Pin, Connector_PinHeader_2.54mm:PinHeader_1x04_P2.54mm_Vertical, F.Cu at (147.2, 89.9)
- added D1: ~, Package_TO_SOT_THT:TO-18-2_Window, F.Cu at (175.5, 73.1)
- added D2: ~, Package_TO_SOT_THT:TO-18-2_Window, F.Cu at (175.5, 80.8)
- added D3: ~, Package_TO_SOT_THT:TO-18-2_Window, F.Cu at (175.5, 88.5)
- added SCREEN1: Conn_01x04_Pin, Connector_PinHeader_2.54mm:PinHeader_1x04_P2.54mm_Vertical, F.Cu at (182.7, 71.3)
- added TOF1: Conn_01x04_Pin, Connector_PinHeader_2.54mm:PinHeader_1x04_P2.54mm_Vertical, F.Cu at (147.2, 87.4)
- added TOF2: Conn_01x04_Pin, Connector_PinHeader_2.54mm:PinHeader_1x04_P2.54mm_Vertical, F.Cu at (147.2, 92.5)
- added TOF3: Conn_01x04_Pin, Connector_PinHeader_2.54mm:PinHeader_1x04_P2.54mm_Vertical, F.Cu at (147.2, 95.0)
Connections:
- net /VCC_5V renamed VCC_5V
- U1 pad 10: unconnected-(U1-IO17-Pad10) -> SDA
- U1 pad 11: unconnected-(U1-IO18-Pad11) -> SCL
Other:
- board text removed: "DRIVER 4"
