File: _autosave-PCB.kicad_pcb (KiCad board)
At the start: 2 copper layers, 60 x 60 mm, 54 parts, among them J1 USB_C_Receptacle_USB2.0_16P, J10 Conn_01x05_Pin, J11 Conn_01x05_Pin, J12 Conn_01x03_Pin, J3 Conn_01x04_Pin, J5 Conn_01x02_Pin, J6 Conn_01x02_Pin, J7 Conn_01x02_Pin, J8 Conn_01x04_Pin, SW1 SW_Push, SW2 SW_Push, U1 TMC2209_SILENTSTEPSTICK, U3 D3V3XA4B10LP, U4 AMS1117-3.3 (UMW), U5 TMC2209_SILENTSTEPSTICK, U6 ESP32-S3-WROOM-1

Commit message: V2 avec test DRC OK
Routing:
- net (no net): vias 2 -> 0
Changed lines of the file:
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@@
 		)
-	)
-	(via
-		(at 167.2 76)
-		(size 0.6)
-		(drill 0.3)
-		(layers "F.Cu" "B.Cu")
-		(net 0)
-	)
-	(via
-		(at 167.2 76)
-		(size 0.6)
-		(drill 0.3)
-		(layers "F.Cu" "B.Cu")
-		(net 0)
 	)
 	(segment
