File: PCB.kicad_pcb (KiCad board)
At the start: 2 copper layers, 60 x 60 mm, 52 parts, among them J1 USB_C_Receptacle_USB2.0_16P, J10 Conn_01x06_Socket, J11 Conn_01x02_Pin, J13 Conn_01x05_Pin, J2 Conn_01x06_Socket, J3 Conn_01x04_Pin, J4 Conn_01x05_Pin, J5 Conn_01x02_Pin, J6 Conn_01x02_Pin, J7 Conn_01x02_Pin, J8 Conn_01x04_Pin, J9 Conn_01x05_Pin, SW1 SW_Push, SW2 SW_Push, U1 TMC2209_SILENTSTEPSTICK, U2 USBLC6-2SC6, U4 AMS1117-3.3 (UMW), U5 TMC2209_SILENTSTEPSTICK, U6 ESP32-S3-WROOM-1

Commit message: suppression C boot + ajout R boot
Parts:
- removed C1: 0.1uF, Capacitor_SMD:C_0805_2012Metric_Pad1.18x1.45mm_HandSolder
- added R10: 10k, Resistor_SMD:R_1206_3216Metric_Pad1.30x1.75mm_HandSolder, F.Cu at (122.2, 128.3)
- C2: value 0.1uF -> 10uF
- moved SW1 0.90 mm to (127.1, 129.3)
Routing:
- net 3V3: track 221.0 -> 223.9 mm
- net BOOT: track 25.4 -> 24.8 mm
- net GND: vias 191 -> 189
Other:
- board text added: "BOOT"
- board text added: "R220"
- board text added: "RST"
